File: HandheldProject.kicad_sch (KiCad schematic)
At the start: 1 part, among them J1 Raspberry_Pi_2_3

Commit message: My Board works in the 3D thing
Parts:
- added BT1: Battery_Cell, Battery:BatteryHolder_Keystone_1060_1x2032, symbol Device:Battery_Cell
- J1: footprint (none) -> Module:Raspberry_Pi_Zero_Socketed_THT_FaceDown_MountingHoles
Connections:
- net GND: now reaches J1.14 (GND), J1.20 (GND), J1.25 (GND), J1.30 (GND), J1.34 (GND), J1.39 (GND), J1.6 (GND), J1.9 (GND)
- net GND: now also BT1.2 (-)
- net +5V: now reaches J1.2 (5V), J1.4 (5V)
- net +5V: now also BT1.1 (+)

Commit message: I hope this doesn't mess up my footprints
Parts:
- removed BT1: Battery_Cell, Battery:BatteryHolder_Keystone_1060_1x2032, symbol Device:Battery_Cell
- removed J1: Raspberry_Pi_2_3, Module:Raspberry_Pi_Zero_Socketed_THT_FaceDown_MountingHoles, symbol Connector:Raspberry_Pi_2_3

Commit message: Just added title. About to move Symbol location out of HandheldSymbols and delete it completely
Other:
- title: (none) -> Handheld_PCB
Changed lines of the file:
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@@
 	(generator_version "8.0")
 	(paper "A4")
+	(title_block
+		(title "Handheld_PCB")
+		(date "2024-12-27")
+		(rev "1.0")
+	)
 	(sheet_instances
 		(path "/"
