File: HandheldProject.kicad_sch (KiCad schematic)
At the start: 0 parts

Commit message: I brought the symbol to the main folder
Parts:
- added Raspberry_Pi_Zero_2_W_For_Schematic1: ~, symbol GitHubTest_Raspberry_Pi_Zero_2_W_Library:Raspberry_Pi_Zero_2_W_Symbol
Connections:
- new net +3.3V: Raspberry_Pi_Zero_2_W_For_Schematic1.0 (3.3V)
Changed lines of the file:
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@@
 	(generator_version "8.0")
 	(paper "A4")
+	(wire
+		(pts
+			(xy 142.24 81.28) (xy 114.3 81.28)
+		)
+		(stroke
+			(width 0)
+			(type default)
+		)
+	)
+	(wire
+		(pts
+			(xy 114.3 81.28) (xy 114.3 77.47)
+		)
+		(stroke
+			(width 0)
+			(type default)
+		)
+	)
+	(symbol
+		(lib_id "GitHubTest_Raspberry_Pi_Zero_2_W_Library:Raspberry_Pi_Zero_2_W_Symbol")
+		(at 173.99 97.79 0)
+		(unit 1)
+		(exclude_from_sim no)
+		(in_bom yes)
+		(on_board yes)
+		(dnp no)
+		(fields_autoplaced yes)
+		(property "Reference" "Raspberry_Pi_Zero_2_W_For_Schematic1"
+			(at 175.895 76.2 0)
+			(effects
+				(font
+					(size 1.27 1.27)
+				)
+			)
+		)
+		(property "Value" "~"
+			(at 175.895 78.74 0)
+			(effects
+				(font
+					(size 1.27 1.27)
+				)
+			)
+		)
+		(property "Footprint" ""
+			(at 173.99 97.79 0)
+			(effects
+				(font
+					(size 1.27 1.27)
+				)
+				(hide yes)
+			)
+		)
+		(property "Datasheet" ""
+			(at 173.99 97.79 0)
+			(effects
+				(font
+					(size 1.27 1.27)
+				)
+				(hide yes)
+			)
+		)
+		(property "Description" ""
+			(at 173.99 97.79 0)
+			(effects
+				(font
+					(size 1.27 1.27)
+				)
+				(hide yes)
+			)
+		)
+		(pin "1"
+		)
+		(pin "12"
+		)
+		(pin "13"
+		)
+		(pin "0"
+		)
+		(pin "14"
+		)
+		(pin "10"
+		)
+		(pin "15"
+		)
+		(pin "16"
+		)
+		(pin "17"
+		)
+		(pin "18"
+		)
+		(pin "11"
+		)
+		(pin "27"
+		)
+		(pin "6"
+		)
+		(pin "20"
+		)
+		(pin "25"
+		)
+		(pin "5"
+		)
+		(pin "7"
+		)
+		(pin "36"
+		)
+		(pin "8"
+		)
+		(pin "9"
+		)
+		(pin "2"
+		)
+		(pin "19"
+		)
+		(pin "29"
+		)
+		(pin "22"
+		)
+		(pin "34"
+		)
+		(pin "21"
+		)
+		(pin "39"
+		)
+		(pin "26"
+		)
+		(pin "23"
+		)
+		(pin "35"
+		)
+		(pin "38"
+		)
+		(pin "4"
+		)
+		(pin "37"
+		)
+		(pin "33"
+		)
+		(pin "3"
+		)
+		(pin "28"
+		)
+		(pin "30"
+		)
+		(pin "32"
+		)
+		(pin "24"
+		)
+		(pin "31"
+		)
+		(instances
+			(project ""
+				(path "/bd82f029-59b3-47bf-a2cf-764bce05225c"
+					(reference "Raspberry_Pi_Zero_2_W_For_Schematic1")
+					(unit 1)
+				)
+			)
+		)
+	)
+	(symbol
+		(lib_id "power:+3.3V")
+		(at 114.3 77.47 0)
+		(unit 1)
+		(exclude_from_sim no)
+		(in_bom yes)
+		(on_board yes)
+		(dnp no)
+		(fields_autoplaced yes)
+		(property "Reference" "#PWR01"
+			(at 114.3 81.28 0)
+			(effects
+				(font
+					(size 1.27 1.27)
+				)
+				(hide yes)
+			)
+		)
+		(property "Value" "+3.3V"
+			(at 114.3 72.39 0)
+			(effects
+				(font
+					(size 1.27 1.27)
+				)
+			)
+		)
+		(property "Footprint" ""
+			(at 114.3 77.47 0)
+			(effects
+				(font
+					(size 1.27 1.27)
+				)
+				(hide yes)
+			)
+		)
+		(property "Datasheet" ""
+			(at 114.3 77.47 0)
+			(effects
+				(font
+					(size 1.27 1.27)
+				)
+				(hide yes)
+			)
+		)
+		(property "Description" "Power symbol creates a global label with name \"+3.3V\""
+			(at 114.3 77.47 0)
+			(effects
+				(font
+					(size 1.27 1.27)
+				)
+				(hide yes)
+			)
+		)
+		(pin "1"
+		)
+		(instances
+			(project ""
+				(path "/bd82f029-59b3-47bf-a2cf-764bce05225c"
+					(reference "#PWR01")
+					(unit 1)
+				)
+			)
+		)
+	)
 	(sheet_instances
 		(path "/"

Commit message: I made so many mistakes. I almost got rid of my snake game
Parts:
- removed Raspberry_Pi_Zero_2_W_For_Schematic1: ~, symbol GitHubTest_Raspberry_Pi_Zero_2_W_Library:Raspberry_Pi_Zero_2_W_Symbol
- added R1, R2, R3, R4, R5, R6, R7: 10k, symbol Device:R
- added Raspberry_Pi_Zero_2_W_For_Schematic2: ~, symbol GitHubTest_Raspberry_Pi_Zero_2_W_Library:Raspberry_Pi_Zero_2_W_Symbol
- added S1, S2, S3, S4: ~, symbol 4_Pin_Push_Button_Switch_Library:4_Pin_Push_Button_Switch
- added S5, S6, S7: ~, symbol Shakir_Switch_Library:Right_Angle_Switch
- added U1: ~, symbol Shakir_Display_Library:TFT_LCD_3.2_inch_(ILI9341)
Connections:
- net +3.3V: now also R1.1, R2.1, R3.1, R4.1, R5.1, R6.1, R7.1, Raspberry_Pi_Zero_2_W_For_Schematic2.0 (3.3V)
- new net: R1.2, S1.1
- new net: R4.2, S4.1
- new net: R2.2, S2.1
- new net: R6.2, S6.1
- new net: R5.2, S5.1
- new net: R3.2, S3.1
- new net: R7.2, S7.1
- new net +5V: Raspberry_Pi_Zero_2_W_For_Schematic2.20 (5V), Raspberry_Pi_Zero_2_W_For_Schematic2.21 (5V)
- new net A (Button): Raspberry_Pi_Zero_2_W_For_Schematic2.7 (GPIO_22), S3.3
- new net B (Button): Raspberry_Pi_Zero_2_W_For_Schematic2.27 (GPIO_23), S4.3
- new net BCK: Raspberry_Pi_Zero_2_W_For_Schematic2.25 (GPIO_18_Chip_Enable-CE0_(SP1)_[PWM])
- new net CSX: Raspberry_Pi_Zero_2_W_For_Schematic2.31 (GPIO_8_Chip_Enable-CE0_(SPI0))
- new net DIN: Raspberry_Pi_Zero_2_W_For_Schematic2.39 (GPIO_21_SCLK_(SPI_1))
- new net DOWN: Raspberry_Pi_Zero_2_W_For_Schematic2.6 (GPIO_27)
- new net D/CX: Raspberry_Pi_Zero_2_W_For_Schematic2.28 (GPIO_24)
- new net GND: Raspberry_Pi_Zero_2_W_For_Schematic2.19 (Ground), Raspberry_Pi_Zero_2_W_For_Schematic2.34 (Ground), Raspberry_Pi_Zero_2_W_For_Schematic2.36 (Ground), S1.2, S2.2, S3.2, S4.2, S5.2, S6.2, S7.2
- new net L (Button): Raspberry_Pi_Zero_2_W_For_Schematic2.15 (GPIO_6), S5.3
- new net LCK: Raspberry_Pi_Zero_2_W_For_Schematic2.17 ([PWM]_GPIO_19_MISO_(SPI_1))
- new net LEFT: Raspberry_Pi_Zero_2_W_For_Schematic2.3 (GPIO_4)
- new net R (Button): Raspberry_Pi_Zero_2_W_For_Schematic2.35 (GPIO_12_(PWM)), S6.3
- new net RESET: Raspberry_Pi_Zero_2_W_For_Schematic2.30 (GPIO_25), U1.4 (RESET)
- new net RIGHT: Raspberry_Pi_Zero_2_W_For_Schematic2.5 (GPIO_17_Chip_Enable-CE1_(SPI1))
- new net SCL: Raspberry_Pi_Zero_2_W_For_Schematic2.11 (GPIO_11_SCLK_(SPI_0))
- new net SDI: Raspberry_Pi_Zero_2_W_For_Schematic2.9 (GPIO_10_MOSI_(SPI_0))
- new net SDO: Raspberry_Pi_Zero_2_W_For_Schematic2.10 (GPIO_09_MISO_(SPI_0))
- new net SELECT: Raspberry_Pi_Zero_2_W_For_Schematic2.37 (GPIO_16_Chip_Enable-CE2_(SPI_1))
- new net START: Raspberry_Pi_Zero_2_W_For_Schematic2.16 (GPIO_13_(PWM))
- new net UP: Raspberry_Pi_Zero_2_W_For_Schematic2.24 (GPIO_15_(UART_RX))
- new net X (Button): Raspberry_Pi_Zero_2_W_For_Schematic2.1 (GPIO_2_Serial_Data_I2C), S1.3
- new net Y (Button): Raspberry_Pi_Zero_2_W_For_Schematic2.2 (GPIO3_Serial_Clock_I2C), S2.3
- new net Z/System (Button): Raspberry_Pi_Zero_2_W_For_Schematic2.14 (GPIO_5), S7.3
- no-connect marks 0 -> 19
Other:
- note added: "Fix me just in case"
- note added: "Need: Raspeberry Pi (check), 4 ABXY Buttons, 4 D-Pad Directional Inputs, System Button (I don't think there is a Start and Select button), L and R buttons (I don't think I have enough for ZR and ZL), Switch for ON and OFf, Switch for Audio and Mute, I don't know what else"
